Commit message: Add one-drone full autonomy deployment stack

File: Autonomy/slam_package/slam/urdf/drone.urdf (robot description, URDF)
Before this commit: robot drone, 5 links, 4 joints
Links:
- added link camera_left_optical_frame
- added link camera_right_optical_frame
Joints:
- added joint camera_left_to_optical: type fixed, parent camera_left_frame, child camera_left_optical_frame, origin xyz=0 0 0 rpy=-1.57079632679 0 -1.57079632679
- added joint camera_right_to_optical: type fixed, parent camera_right_frame, child camera_right_optical_frame, origin xyz=0 0 0 rpy=-1.57079632679 0 -1.57079632679
- joint base_to_camera_left: origin xyz=0 0.05 0 rpy=0 0 0 -> xyz=0 0.0289816 0 rpy=0 0 0
- joint base_to_camera_right: origin xyz=0 -0.05 0 rpy=0 0 0 -> xyz=0 -0.0289816 0 rpy=0 0 0
